Commit message: Removed files Unnecesary files from forked repo

File: enviroment/knife.urdf (robot description, URDF)
Before this commit: robot cube.urdf, 1 links, 0 joints
Links:
- link baseLink: geometry collision mesh filename=cup.obj scale=0.5 0.5 0.5; visual mesh filename=cup.obj scale=0.5 0.5 0.5
